File: Eagle/larrow.sch (EAGLE design)
At the start: 39 parts, among them T1 2N2222, T10 2N2222, T11 2N2222, T12 2N2222, T2 2N2222, T3 2N2222, T4 2N2222, T5 2N2222, T6 2N2222, T7 2N2222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

Commit message: Added label
Other:
- note added: "Launchpad powered via USB"
Changed lines of the file:
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@@
 <sheet>
 <plain>
+<text x="172.72" y="73.66" size="1.778" layer="91">Launchpad powered via USB</text>
 </plain>
 <instances>
